File: pcb/kasumigasane-plate3.kicad_pcb (KiCad board)
At the start: 2 copper layers, 90 x 90 mm, 49 parts

Commit message: remove mousebites
Parts:
- removed the ? at (102.0, 66.5)
- removed the ? at (68.0, 66.5)
- removed the ? at (38.5, 66.5)
- removed the ? at (31.0, 66.5)
- removed the ? at (75.5, 66.5)
- removed the ? at (28.5, 66.5)
- removed the ? at (65.0, 66.5)
- removed the ? at (94.5, 66.5)
- removed the ? at (57.5, 66.5)
- removed the ? at (104.5, 66.5)
