File: pcb/kasumigasane-plate4.kicad_pcb (KiCad board)
At the start: 2 copper layers, 90 x 90 mm, 56 parts

Commit message: remove mousebites
Parts:
- removed the ? at (37.0, 66.5)
- removed the ? at (70.0, 66.5)
- removed the ? at (103.5, 66.5)
- removed the ? at (28.5, 66.5)
- removed the ? at (96.0, 66.5)
- removed the ? at (51.0, 65.0)
- removed the ? at (29.5, 66.5)
- removed the ? at (104.5, 66.5)
- removed the ? at (71.0, 66.5)
- removed the ? at (62.5, 66.5)
- removed the ? at (51.0, 64.0)
- removed the ? at (78.5, 66.5)
